File: launcher/schematics/pepermoot.kicad_pcb (KiCad board)
At the start: 2 copper layers, 18 parts, among them J1 Pull motor, J2 End switch, J3 Power, J4 Dispenser motor, J5 Servo, J6 Pull motor, J7 Extra, U2 ESP32-DevKitC

Commit message: pcb update
Parts:
- moved J6 96.0 mm to (111.0, 35.0), turned to -90 degrees
- moved J5 87.9 mm to (68.5, 138.3), turned to 180 degrees
- moved J2 87.7 mm to (59.0, 97.5), turned to 90 degrees
- moved J1 82.6 mm to (89.5, 137.0)
- moved J4 73.2 mm to (111.0, 46.0), turned to -90 degrees
- moved R4 71.6 mm to (113.0, 70.0), turned to 180 degrees
- moved C1 68.8 mm to (137.0, 142.6), turned to -90 degrees
- moved J3 65.0 mm to (107.0, 137.0)
- moved A1 64.3 mm to (89.3, 62.4), turned to 180 degrees
- moved C2 63.7 mm to (122.0, 143.0), turned to -90 degrees
- moved J7 58.1 mm to (111.0, 78.0), turned to -90 degrees
- moved R1 49.5 mm to (114.8, 93.0), turned to 180 degrees
- moved R2 47.8 mm to (114.8, 100.0), turned to 180 degrees
- moved R3 46.3 mm to (115.0, 107.0), turned to 180 degrees
- moved D1 44.6 mm to (124.9, 93.0)
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Connections:
- J5 pad 1: GND -> +5V
- J5 pad 2: +5V -> GND
Routing:
- net GND: track 0.00 -> 500.1 mm
- net Net-(A1-M0): track 0.00 -> 239.7 mm
- net +24V: track 0.00 -> 192.9 mm
- net +5V: track 0.00 -> 97.4 mm
- net Net-(J5-Pin_3): track 0.00 -> 63.4 mm
- net Net-(A1-~{EN}): track 0.00 -> 61.0 mm
- net Net-(J1-Pin_3): track 0.00 -> 60.5 mm
- net Net-(A1-DIR): track 0.00 -> 43.9 mm
- net Net-(A1-STEP): track 0.00 -> 43.5 mm
- net Net-(J1-Pin_1): track 0.00 -> 40.2 mm
- net Net-(A1-A2): track 0.00 -> 37.4 mm
- net Net-(J1-Pin_2): track 0.00 -> 34.9 mm
- net Net-(A1-B2): track 0.00 -> 23.2 mm
- net Net-(A1-B1): track 0.00 -> 23.2 mm
- net Net-(A1-A1): track 0.00 -> 22.1 mm
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
Commit message: Move resistor
Parts:
- moved R4 46.9 mm to (78.2, 38.5), turned to 0 degrees
Routing:
- net Net-(A1-~{EN}): track 61.0 -> 58.7 mm
- net Net-(A1-M0): track 239.7 -> 240.8 mm
Changed lines of the file:
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@@
 	(footprint "Resistor_THT:R_Axial_DIN0204_L3.6mm_D1.6mm_P7.62mm_Horizontal"
 		(layer "F.Cu")
-		(at 113 70 180)
+		(at 78.19 38.5)
 		(descr "Resistor, Axial_DIN0204 series, Axial, Horizontal, pin pitch=7.62mm, 0.167W, length*diameter=3.6*1.6mm^2, http://cdn-reichelt.de/documents/datenblatt/B400/1_4W%23YAG.pdf")
 		(tags "Resistor Axial_DIN0204 series Axial Horizontal pin pitch 7.62mm 0.167W length 3.6mm diameter 1.6mm")
@@
 		(duplicate_pad_numbers_are_jumpers no)
 		(fp_line
-			(start 6.68 0)
-			(end 5.73 0)
+			(start 0.94 0)
+			(end 1.89 0)
 			(stroke
 				(width 0.12)
@@
 		)
 		(fp_line
-			(start 0.94 0)
-			(end 1.89 0)
+			(start 6.68 0)
+			(end 5.73 0)
 			(stroke
 				(width 0.12)
@@
 		)
 		(fp_line
-			(start 7.62 0)
-			(end 5.61 0)
+			(start 0 0)
+			(end 2.01 0)
 			(stroke
 				(width 0.1)
@@
 		)
 		(fp_line
-			(start 0 0)
-			(end 2.01 0)
+			(start 7.62 0)
+			(end 5.61 0)
 			(stroke
 				(width 0.1)
@@
 		)
 		(pad "1" thru_hole circle
-			(at 0 0 180)
+			(at 0 0)
 			(size 1.4 1.4)
 			(drill 0.7)
@@
 		)
 		(pad "2" thru_hole circle
-			(at 7.62 0 180)
+			(at 7.62 0)
 			(size 1.4 1.4)
 			(drill 0.7)
@@
 	)
 	(segment
+		(start 73 40)
+		(end 74.5 38.5)
+		(width 1)
+		(layer "B.Cu")
+		(net "Net-(A1-M0)")
+	)
+	(segment
 		(start 65 57)
 		(end 65 24)
@@
 	)
 	(segment
+		(start 74.15 47.15)
+		(end 73 46)
+		(width 1)
+		(layer "B.Cu")
+		(net "Net-(A1-M0)")
+	)
+	(segment
 		(start 65.31 57.31)
 		(end 65 57)
@@
 	)
 	(segment
+		(start 73 46)
+		(end 73 40)
+		(width 1)
+		(layer "B.Cu")
+		(net "Net-(A1-M0)")
+	)
+	(segment
 		(start 127.465 93)
 		(end 127.465 71)
@@
 	)
 	(segment
+		(start 74.5 38.5)
+		(end 78.19 38.5)
+		(width 1)
+		(layer "B.Cu")
+		(net "Net-(A1-M0)")
+	)
+	(segment
 		(start 65 76)
 		(end 65 57)
@@
 	)
 	(segment
-		(start 126.465 70)
-		(end 127.465 71)
-		(width 1)
-		(layer "B.Cu")
-		(net "Net-(A1-M0)")
-	)
-	(segment
-		(start 113 70)
-		(end 126.465 70)
+		(start 76.64 47.15)
+		(end 76.64 49.69)
 		(width 1)
 		(layer "B.Cu")
@@
 	(segment
 		(start 76.64 47.15)
-		(end 76.64 49.69)
+		(end 74.15 47.15)
 		(width 1)
 		(layer "B.Cu")
@@
 	)
 	(segment
-		(start 80.61 44.61)
+		(start 79.5 44.61)
+		(end 82.89 44.61)
+		(width 1)
+		(layer "B.Cu")
+		(net "Net-(A1-~{EN})")
+	)
+	(segment
+		(start 83 44.5)
+		(end 85.81 41.69)
+		(width 1)
+		(layer "B.Cu")
+		(net "Net-(A1-~{EN})")
+	)
+	(segment
+		(start 79.5 44.61)
 		(end 76.64 44.61)
 		(width 1)
@@
 	)
 	(segment
+		(start 83 72)
+		(end 83 44.5)
+		(width 1)
+		(layer "B.Cu")
+		(net "Net-(A1-~{EN})")
+	)
+	(segment
 		(start 96.5 78.54)
 		(end 96.84 78.54)
@@
 	)
 	(segment
-		(start 83 47)
-		(end 80.61 44.61)
+		(start 82.89 44.61)
+		(end 83 44.5)
 		(width 1)
 		(layer "B.Cu")
@@
 	)
 	(segment
-		(start 96.84 78.54)
-		(end 105.38 70)
+		(start 85.81 41.69)
+		(end 85.81 38.5)
 		(width 1)
 		(layer "B.Cu")
@@
 	)
 	(segment
-		(start 89.54 78.54)
-		(end 83 72)
+		(start 80.61 44.61)
+		(end 79.5 44.61)
 		(width 1)
 		(layer "B.Cu")
@@
 	)
 	(segment
-		(start 83 72)
-		(end 83 47)
+		(start 89.54 78.54)
+		(end 83 72)
 		(width 1)
 		(layer "B.Cu")

Commit message: pcb update
Parts:
- removed J1: Pull motor, TerminalBlock:TerminalBlock_Xinya_XY308-2.54-3P_1x03_P2.54mm_Horizontal
- removed J2: End switch, TerminalBlock:TerminalBlock_Xinya_XY308-2.54-2P_1x02_P2.54mm_Horizontal
- removed J5: Servo, TerminalBlock:TerminalBlock_Xinya_XY308-2.54-3P_1x03_P2.54mm_Horizontal
- removed J6: Pull motor, TerminalBlock:TerminalBlock_Xinya_XY308-2.54-2P_1x02_P2.54mm_Horizontal
- added J8: Pul motor, TerminalBlock:TerminalBlock_Xinya_XY308-2.54-5P_1x05_P2.54mm_Horizontal, F.Cu at (100.8, 133.0)
- added J9: End switch (1,2) , Servo (3,4,5), TerminalBlock:TerminalBlock_Xinya_XY308-2.54-5P_1x05_P2.54mm_Horizontal, F.Cu at (57.0, 133.0)
- R1, R2, R3: footprint Resistor_THT:R_Axial_DIN0204_L3.6mm_D1.6mm_P7.62mm_Horizontal -> Resistor_THT:R_Axial_DIN0207_L6.3mm_D2.5mm_P10.16mm_Horizontal
- moved C1 103.9 mm to (96.5, 47.0), turned to 0 degrees
- moved C2 24.6 mm to (127.4, 119.0), turned to 180 degrees
- moved J3 14.1 mm to (120.5, 133.0)
- moved J4 13.8 mm to (120.5, 56.0)
- moved J7 10.3 mm to (120.5, 74.0)
Routing:
- net Net-(A1-M0): track 240.8 -> 187.7 mm
- net Net-(J9-Pin_2): track 13.7 -> 51.2 mm
- net GND: track 500.1 -> 463.0 mm
- net +24V: track 192.9 -> 166.4 mm
- net Net-(J9-Pin_3): track 63.4 -> 46.7 mm
- net +5V: track 97.4 -> 112.2 mm
- net Net-(A1-A2): track 37.4 -> 50.7 mm
- net Net-(A1-A1): track 22.1 -> 34.8 mm
- net Net-(J8-Pin_3): track 60.5 -> 71.8 mm
- net Net-(J7-Pin_1): track 15.8 -> 26.9 mm
- net Net-(J7-Pin_3): track 16.9 -> 28.1 mm
- net Net-(A1-B2): track 23.2 -> 33.8 mm
- net Net-(A1-B1): track 23.2 -> 33.8 mm
- net Net-(J8-Pin_2): track 34.9 -> 40.3 mm
- net Net-(J8-Pin_1): track 40.2 -> 43.2 mm
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
Commit message: pcb update
Parts:
- added REF**: MountingHole_3.2mm_M3, MountingHole:MountingHole_3.2mm_M3, F.Cu at (56.0, 36.0)
- added REF**: MountingHole_3.2mm_M3, MountingHole:MountingHole_3.2mm_M3, F.Cu at (131.0, 36.0)
- added REF**: MountingHole_3.2mm_M3, MountingHole:MountingHole_3.2mm_M3, F.Cu at (56.0, 146.0)
- added REF**: MountingHole_3.2mm_M3, MountingHole:MountingHole_3.2mm_M3, F.Cu at (131.0, 146.0)
Routing:
- net GND: track 463.0 -> 456.7 mm
- net Net-(A1-M0): track 187.7 -> 186.3 mm
- net +5V: track 112.2 -> 111.0 mm
- net +24V: track 166.4 -> 165.6 mm
Other:
- board outline added: 83 x 119 mm

Commit message: Minor update
Parts:
- moved R4 1.69 mm to (79.9, 38.5)
Routing:
- net GND: track 456.7 -> 455.2 mm
- net +24V: track 165.6 -> 164.3 mm
- net Net-(A1-~{EN}): track 59.6 -> 60.8 mm
Changed lines of the file:
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@@
 	(footprint "Resistor_THT:R_Axial_DIN0204_L3.6mm_D1.6mm_P7.62mm_Horizontal"
 		(layer "F.Cu")
-		(at 78.19 38.5)
+		(at 79.88 38.5)
 		(descr "Resistor, Axial_DIN0204 series, Axial, Horizontal, pin pitch=7.62mm, 0.167W, length*diameter=3.6*1.6mm^2, http://cdn-reichelt.de/documents/datenblatt/B400/1_4W%23YAG.pdf")
 		(tags "Resistor Axial_DIN0204 series Axial Horizontal pin pitch 7.62mm 0.167W length 3.6mm diameter 1.6mm")
@@
 			(at 3.81 -1.92 0)
 			(layer "F.SilkS")
+			(hide yes)
 			(effects
 				(font
@@
 		)
 		(fp_text user "${REFERENCE}"
-			(at 3.81 0 0)
+			(at 6.68 0 0)
 			(layer "F.Fab")
 			(effects
@@
 	)
 	(segment
-		(start 74.5 38.5)
-		(end 78.19 38.5)
-		(width 1.5)
-		(layer "B.Cu")
-		(net "Net-(A1-M0)")
-	)
-	(segment
 		(start 131 89.465)
 		(end 131 48.5)
@@
 	)
 	(segment
-		(start 81.5 35.5)
-		(end 78.5 38.5)
-		(width 1.5)
-		(layer "B.Cu")
-		(net "Net-(A1-M0)")
-	)
-	(segment
-		(start 78.5 38.5)
-		(end 78.19 38.5)
-		(width 1.5)
-		(layer "B.Cu")
-		(net "Net-(A1-M0)")
-	)
-	(segment
-		(start 118 35.5)
-		(end 81.5 35.5)
+		(start 68 47)
+		(end 68 40.5)
 		(width 1.5)
 		(layer "B.Cu")
@@
 	)
 	(segment
-		(start 68 47)
-		(end 68 40.5)
+		(start 68 72.9)
+		(end 68 47)
 		(width 1.5)
 		(layer "B.Cu")
@@
 	)
 	(segment
-		(start 68 72.9)
-		(end 68 47)
+		(start 76.64 47.15)
+		(end 76.64 49.69)
 		(width 1.5)
 		(layer "B.Cu")
@@
 	)
 	(segment
-		(start 70 38.5)
-		(end 74.5 38.5)
+		(start 76.64 52.23)
+		(end 76.64 54.77)
 		(width 1.5)
 		(layer "B.Cu")
@@
 	)
 	(segment
-		(start 76.64 47.15)
-		(end 76.64 49.69)
+		(start 82.88 35.5)
+		(end 79.88 38.5)
 		(width 1.5)
 		(layer "B.Cu")
@@
 	)
 	(segment
-		(start 76.64 52.23)
-		(end 76.64 54.77)
+		(start 127.465 93)
+		(end 131 89.465)
 		(width 1.5)
 		(layer "B.Cu")
@@
 	)
 	(segment
-		(start 127.465 93)
-		(end 131 89.465)
+		(start 70 38.5)
+		(end 79.88 38.5)
 		(width 1.5)
 		(layer "B.Cu")
@@
 	)
 	(segment
-		(start 79.5 44.61)
-		(end 82.89 44.61)
-		(width 1.5)
-		(layer "B.Cu")
-		(net "Net-(A1-~{EN})")
-	)
-	(segment
-		(start 83 44.5)
-		(end 85.81 41.69)
+		(start 118 35.5)
+		(end 82.88 35.5)
 		(width 1.5)
 		(layer "B.Cu")
-		(net "Net-(A1-~{EN})")
+		(net "Net-(A1-M0)")
 	)
 	(segment
@@
 	)
 	(segment
-		(start 79.5 44.61)
+		(start 78.89 44.61)
 		(end 76.64 44.61)
 		(width 1.5)
@@
 	)
 	(segment
-		(start 82 45.5)
-		(end 83 44.5)
+		(start 96.5 78.54)
+		(end 96.84 78.54)
 		(width 1.5)
 		(layer "B.Cu")
@@
 	)
 	(segment
-		(start 96.5 78.54)
-		(end 96.84 78.54)
+		(start 82 71)
+		(end 82 44)
 		(width 1.5)
 		(layer "B.Cu")
@@
 	)
 	(segment
-		(start 82.89 44.61)
-		(end 83 44.5)
+		(start 96.5 78.54)
+		(end 89.54 78.54)
 		(width 1.5)
 		(layer "B.Cu")
@@
 	)
 	(segment
-		(start 96.5 78.54)
-		(end 89.54 78.54)
+		(start 82 44)
+		(end 87.5 38.5)
 		(width 1.5)
 		(layer "B.Cu")
@@
 	)
 	(segment
-		(start 85.81 41.69)
-		(end 85.81 38.5)
+		(start 79 44.5)
+		(end 78.89 44.61)
 		(width 1.5)
 		(layer "B.Cu")
@@
 	)
 	(segment
-		(start 80.61 44.61)
-		(end 79.5 44.61)
+		(start 76.64 44.61)
+		(end 81.39 44.61)
 		(width 1.5)
 		(layer "B.Cu")
@@
 	)
 	(segment
-		(start 82 71)
-		(end 82 45.5)
+		(start 81.39 44.61)
+		(end 82 44)
 		(width 1.5)
 		(layer "B.Cu")
@@
 	)
 	(segment
-		(start 89.34 47.15)
-		(end 90.85 47.15)
-		(width 1.5)
-		(layer "B.Cu")
-		(net "GND")
-	)
-	(segment
 		(start 107 141.5)
 		(end 80.5 141.5)
@@
 	)
 	(segment
-		(start 112 91)
-		(end 112.08 91.08)
-		(width 1.5)
-		(layer "B.Cu")
-		(net "+24V")
-	)
-	(segment
 		(start 114.5 133)
 		(end 114.5 137.5)
@@
 	)
 	(segment
-		(start 114.5 122.92)
-		(end 114.5 133)
+		(start 114 89)
+		(end 124.5 89)
 		(width 1.5)
 		(layer "B.Cu")
@@
 	)
 	(segment
-		(start 112.08 91.08)
-		(end 112.08 120.5)
+		(start 114.5 122.92)
+		(end 114.5 133)
 		(width 1.5)
 		(layer "B.Cu")
@@
 	)
 	(segment
+		(start 112.08 90.92)
+		(end 114 89)
+		(width 1.5)
+		(layer "B.Cu")
+		(net "+24V")
+	)
+	(segment
 		(start 96.5 47)
 		(end 96.5 43.46)
@@
 	)
 	(segment
-		(start 113.96 43.46)
-		(end 114 43.5)
+		(start 112.08 120.5)
+		(end 112.08 90.92)
 		(width 1.5)
 		(layer "B.Cu")
@@
 	)
 	(segment
-		(start 96.5 43.46)
-		(end 113.96 43.46)
+		(start 113.96 43.46)
+		(end 114 43.5)
 		(width 1.5)
 		(layer "B.Cu")
@@
 	)
 	(segment
-		(start 112 89)
-		(end 112 91)
+		(start 96.5 43.46)
+		(end 113.96 43.46)
 		(width 1.5)
 		(layer "B.Cu")
@@
 		(width 1.5)
 		(layer "B.Cu")
-		(net "+24V")
-	)
-	(segment
-		(start 124.5 89)
-		(end 112 89)
-		(width 1.5)
-		(layer "B.Cu")
