File: launcher/schematics/pepermoot-spiegelbeeld.kicad_pcb (KiCad board)
At the start: 2 copper layers, 83 x 119 mm, 20 parts, among them J3 Power, J4 Dispenser motor, J7 Extra, J8 Pul motor, J9 End switch (1,2) , Servo (3,4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, U2 ESP32-DevKitC

Commit message: pcb update
Parts:
- A1, C1, C2, D1, D2, D3, J3, J4, J7, J8, J9, R1, R2, R3, R4, REF** (x4), U2: moved to B.Cu
- moved REF** 75.0 mm to (131.0, 36.0), turned to 180 degrees
- moved REF** 75.0 mm to (56.0, 36.0), turned to 180 degrees
- moved REF** 75.0 mm to (131.0, 146.0), turned to 180 degrees
- moved REF** 75.0 mm to (56.0, 146.0), turned to 180 degrees
- moved J9 73.0 mm to (130.0, 133.0), turned to 180 degrees
- moved C2 67.7 mm to (59.6, 119.0), turned to 0 degrees
- moved D1 62.8 mm to (62.1, 93.0), turned to 180 degrees
- moved D2 62.8 mm to (62.1, 100.0), turned to 180 degrees
- moved D3 62.8 mm to (62.1, 107.2), turned to 180 degrees
- moved J3 54.0 mm to (66.5, 133.0), turned to 180 degrees
- moved J4 54.0 mm to (66.5, 56.0)
- moved J7 54.0 mm to (66.5, 74.0)
- moved U2 44.8 mm to (115.9, 76.0), turned to 180 degrees
- moved R3 43.0 mm to (72.0, 107.0), turned to 0 degrees
- moved R1 42.6 mm to (72.2, 93.0), turned to 0 degrees
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