File: launcher/schematics/pepermoot.kicad_sch (KiCad schematic)
At the start: 18 parts, among them J1 Pull motor, J2 End switch, J3 Power, J4 Dispenser motor, J5 Servo, J6 Pull motor, J7 Extra, U2 ESP32-DevKitC

Commit message: pcb update
Connections:
- net +5V: now also J5.1 (Pin_1); no longer J5.2 (Pin_2)
- net GND: now also J5.2 (Pin_2); no longer J5.1 (Pin_1)
Other:
- moved on the sheet: C2
Changed lines of the file:
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@@
+	)
+	(junction
+		(at 242.57 125.73)
+		(diameter 0)
+		(color 0 0 0 0)
 	)
 	(junction
@@
 	)
 	(junction
-		(at 236.22 124.46)
-		(diameter 0)
-		(color 0 0 0 0)
-	)
-	(junction
 		(at 97.79 87.63)
 		(diameter 0)
@@
 	)
 	(junction
-		(at 238.76 139.7)
+		(at 242.57 139.7)
 		(diameter 0)
 		(color 0 0 0 0)
@@
 	(wire
 		(pts
-			(xy 236.22 139.7) (xy 238.76 139.7)
-		)
-		(stroke
-			(width 0)
-			(type default)
-		)
-	)
-	(wire
-		(pts
-			(xy 233.68 124.46) (xy 233.68 142.24)
-		)
-		(stroke
-			(width 0)
-			(type default)
-		)
-	)
-	(wire
-		(pts
-			(xy 236.22 124.46) (xy 233.68 124.46)
-		)
-		(stroke
-			(width 0)
-			(type default)
-		)
-	)
-	(wire
-		(pts
 			(xy 82.55 97.79) (xy 82.55 100.33)
 		)
@@
 	(wire
 		(pts
-			(xy 238.76 133.35) (xy 238.76 139.7)
+			(xy 242.57 133.35) (xy 242.57 139.7)
 		)
 		(stroke
@@
 	(wire
 		(pts
+			(xy 236.22 142.24) (xy 236.22 125.73)
+		)
+		(stroke
+			(width 0)
+			(type default)
+		)
+	)
+	(wire
+		(pts
 			(xy 81.28 95.25) (xy 81.28 97.79)
 		)
@@
 	(wire
 		(pts
+			(xy 236.22 125.73) (xy 242.57 125.73)
+		)
+		(stroke
+			(width 0)
+			(type default)
+		)
+	)
+	(wire
+		(pts
 			(xy 97.79 69.85) (xy 97.79 67.31)
 		)
@@
 	(wire
 		(pts
-			(xy 236.22 142.24) (xy 236.22 139.7)
-		)
-		(stroke
-			(width 0)
-			(type default)
-		)
-	)
-	(wire
-		(pts
 			(xy 63.5 29.21) (xy 63.5 31.75)
 		)
@@
 	(wire
 		(pts
-			(xy 238.76 125.73) (xy 238.76 124.46)
-		)
-		(stroke
-			(width 0)
-			(type default)
-		)
-	)
-	(wire
-		(pts
 			(xy 256.54 142.24) (xy 256.54 52.07)
 		)
@@
 	(wire
 		(pts
-			(xy 236.22 121.92) (xy 236.22 124.46)
-		)
-		(stroke
-			(width 0)
-			(type default)
-		)
-	)
-	(wire
-		(pts
 			(xy 135.89 140.97) (xy 135.89 135.89)
 		)
@@
 	(wire
 		(pts
+			(xy 233.68 139.7) (xy 233.68 142.24)
+		)
+		(stroke
+			(width 0)
+			(type default)
+		)
+	)
+	(wire
+		(pts
 			(xy 156.21 72.39) (xy 118.11 72.39)
 		)
@@
 	(wire
 		(pts
-			(xy 238.76 139.7) (xy 242.57 139.7)
-		)
-		(stroke
-			(width 0)
-			(type default)
-		)
-	)
-	(wire
-		(pts
 			(xy 93.98 90.17) (xy 97.79 90.17)
 		)
@@
 	(wire
 		(pts
+			(xy 233.68 139.7) (xy 242.57 139.7)
+		)
+		(stroke
+			(width 0)
+			(type default)
+		)
+	)
+	(wire
+		(pts
 			(xy 186.69 41.91) (xy 186.69 31.75)
 		)
@@
 	(wire
 		(pts
+			(xy 242.57 123.19) (xy 242.57 125.73)
+		)
+		(stroke
+			(width 0)
+			(type default)
+		)
+	)
+	(wire
+		(pts
 			(xy 83.82 97.79) (xy 83.82 95.25)
-		)
-		(stroke
-			(width 0)
-			(type default)
-		)
-	)
-	(wire
-		(pts
-			(xy 238.76 124.46) (xy 236.22 124.46)
 		)
 		(stroke
@@
 	(symbol
 		(lib_id "power:+5V")
-		(at 236.22 121.92 0)
+		(at 242.57 123.19 0)
 		(unit 1)
 		(body_style 1)
@@
 		(fields_autoplaced yes)
 		(property "Reference" "#PWR013"
-			(at 236.22 125.73 0)
+			(at 242.57 127 0)
 			(hide yes)
 			(show_name no)
@@
 		)
 		(property "Value" "+5V"
-			(at 236.22 116.84 0)
+			(at 242.57 118.11 0)
 			(show_name no)
 			(do_not_autoplace no)
@@
 		)
 		(property "Footprint" ""
-			(at 236.22 121.92 0)
+			(at 242.57 123.19 0)
 			(hide yes)
 			(show_name no)
@@
 		)
 		(property "Datasheet" ""
-			(at 236.22 121.92 0)
+			(at 242.57 123.19 0)
 			(hide yes)
 			(show_name no)
@@
 		)
 		(property "Description" "Power symbol creates a global label with name \"+5V\""
-			(at 236.22 121.92 0)
+			(at 242.57 123.19 0)
 			(hide yes)
 			(show_name no)
@@
 	(symbol
 		(lib_id "Device:C_Polarized")
-		(at 238.76 129.54 0)
+		(at 242.57 129.54 0)
 		(unit 1)
 		(body_style 1)
@@
 		(fields_autoplaced yes)
 		(property "Reference" "C2"
-			(at 242.57 127.3809 0)
+			(at 246.38 127.3809 0)
 			(show_name no)
 			(do_not_autoplace no)
@@
 		)
 		(property "Value" "470uF/10V"
-			(at 242.57 129.9209 0)
+			(at 246.38 129.9209 0)
 			(show_name no)
 			(do_not_autoplace no)
@@
 		)
 		(property "Footprint" "Capacitor_THT:CP_Radial_D10.0mm_P5.00mm"
-			(at 239.7252 133.35 0)
+			(at 243.5352 133.35 0)
 			(hide yes)
 			(show_name no)
@@
 		)
 		(property "Datasheet" ""
-			(at 238.76 129.54 0)
+			(at 242.57 129.54 0)
 			(hide yes)
 			(show_name no)
@@
 		)
 		(property "Description" "Polarized capacitor"
-			(at 238.76 129.54 0)
-			(hide yes)
-			(show_name no)
+			(at 242.57 129.54 0)
+			(hide yes)
+			(show_name no)

Commit message: pcb update
Parts:
- removed J1: Pull motor, TerminalBlock:TerminalBlock_Xinya_XY308-2.54-3P_1x03_P2.54mm_Horizontal, symbol Connector:Screw_Terminal_01x03
- removed J2: End switch, TerminalBlock:TerminalBlock_Xinya_XY308-2.54-2P_1x02_P2.54mm_Horizontal, symbol Connector:Screw_Terminal_01x02
- removed J5: Servo, TerminalBlock:TerminalBlock_Xinya_XY308-2.54-3P_1x03_P2.54mm_Horizontal, symbol Connector:Screw_Terminal_01x03
- removed J6: Pull motor, TerminalBlock:TerminalBlock_Xinya_XY308-2.54-2P_1x02_P2.54mm_Horizontal, symbol Connector:Screw_Terminal_01x02
- added J8: Pul motor, TerminalBlock:TerminalBlock_Xinya_XY308-2.54-5P_1x05_P2.54mm_Horizontal, symbol Connector:Screw_Terminal_01x05
- added J9: End switch (1,2) , Servo (3,4,5), TerminalBlock:TerminalBlock_Xinya_XY308-2.54-5P_1x05_P2.54mm_Horizontal, symbol Connector:Screw_Terminal_01x05
- R1, R2, R3: footprint Resistor_THT:R_Axial_DIN0204_L3.6mm_D1.6mm_P7.62mm_Horizontal -> Resistor_THT:R_Axial_DIN0207_L6.3mm_D2.5mm_P10.16mm_Horizontal
Connections:
- net +24V: now also J8.5 (Pin_5)
- net +5V: now also J9.5 (Pin_5)
- net GND: now also J8.4 (Pin_4), J9.1 (Pin_1), J9.4 (Pin_4)
- net at U2.7 (32K_XP/GPIO32/ADC1_CH4): now also J9.2 (Pin_2)
- net at U2.8 (32K_XN/GPIO33/ADC1_CH5): now also J9.3 (Pin_3)
- net at U2.11 (ADC2_CH7/GPIO27): now also J8.3 (Pin_3)
- net at U2.27 (GPIO16): now also J8.2 (Pin_2)
- net at U2.28 (GPIO17): now also J8.1 (Pin_1)

Commit message: pcb update
Other:
- moved on the sheet: C2

Commit message: pcb update
Parts:
- J3: footprint TerminalBlock:TerminalBlock_Xinya_XY308-2.54-3P_1x03_P2.54mm_Horizontal -> TerminalBlock_Phoenix:TerminalBlock_Phoenix_MKDS-1,5-3-5.08_1x03_P5.08mm_Horizontal
- J4: footprint TerminalBlock:TerminalBlock_Xinya_XY308-2.54-4P_1x04_P2.54mm_Horizontal -> TerminalBlock_Phoenix_MKDS-1,5-4-5.08_1x04_P5.08mm_Horizontal
- J7: footprint TerminalBlock:TerminalBlock_Xinya_XY308-2.54-4P_1x04_P2.54mm_Horizontal -> TerminalBlock_Phoenix:TerminalBlock_Phoenix_MKDS-1,5-4-5.08_1x04_P5.08mm_Horizontal
- J8, J9: footprint TerminalBlock:TerminalBlock_Xinya_XY308-2.54-5P_1x05_P2.54mm_Horizontal -> TerminalBlock_Phoenix:TerminalBlock_Phoenix_MKDS-1,5-5-5.08_1x05_P5.08mm_Horizontal
Changed lines of the file:
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@@
 			)
 		)
-		(property "Footprint" "TerminalBlock:TerminalBlock_Xinya_XY308-2.54-4P_1x04_P2.54mm_Horizontal"
+		(property "Footprint" "TerminalBlock_Phoenix_MKDS-1,5-4-5.08_1x04_P5.08mm_Horizontal"
 			(at 68.58 146.05 0)
 			(hide yes)
@@
 			)
 		)
-		(property "Footprint" "TerminalBlock:TerminalBlock_Xinya_XY308-2.54-3P_1x03_P2.54mm_Horizontal"
+		(property "Footprint" "TerminalBlock_Phoenix:TerminalBlock_Phoenix_MKDS-1,5-3-5.08_1x03_P5.08mm_Horizontal"
 			(at 43.18 146.05 0)
 			(hide yes)
@@
 			)
 		)
-		(property "Footprint" "TerminalBlock:TerminalBlock_Xinya_XY308-2.54-5P_1x05_P2.54mm_Horizontal"
+		(property "Footprint" "TerminalBlock_Phoenix:TerminalBlock_Phoenix_MKDS-1,5-5-5.08_1x05_P5.08mm_Horizontal"
 			(at 245.11 158.75 0)
 			(hide yes)
@@
 			)
 		)
-		(property "Footprint" "TerminalBlock:TerminalBlock_Xinya_XY308-2.54-5P_1x05_P2.54mm_Horizontal"
+		(property "Footprint" "TerminalBlock_Phoenix:TerminalBlock_Phoenix_MKDS-1,5-5-5.08_1x05_P5.08mm_Horizontal"
 			(at 143.51 146.05 0)
 			(hide yes)
@@
 			)
 		)
-		(property "Footprint" "TerminalBlock:TerminalBlock_Xinya_XY308-2.54-4P_1x04_P2.54mm_Horizontal"
+		(property "Footprint" "TerminalBlock_Phoenix:TerminalBlock_Phoenix_MKDS-1,5-4-5.08_1x04_P5.08mm_Horizontal"
 			(at 115.57 146.05 0)
 			(hide yes)
