File: schakelbord/schakelbord/schakelbord.kicad_pcb (KiCad board)
At the start: 2 copper layers, 3 parts, among them U1 MCP23017x-x-SP

Commit message: pcb update
Parts:
- removed R1: 10K, PCM_SparkFun-Resistor:R_0603_1608Metric
- added D1: 1N4007, Diode_THT:D_DO-41_SOD81_P10.16mm_Horizontal, F.Cu at (215.0, 23.3)
- added D10: LED, LED_THT:LED_D5.0mm, F.Cu at (74.2, 86.0)
- added D11: LED, LED_THT:LED_D5.0mm, F.Cu at (73.7, 78.5)
- added D12: LED, LED_THT:LED_D5.0mm, F.Cu at (73.7, 71.5)
- added D15: LED, LED_THT:LED_D5.0mm, F.Cu at (75.2, 56.0)
- added D16: LED, LED_THT:LED_D5.0mm, F.Cu at (64.7, 45.0)
- added D17: LED, LED_THT:LED_D5.0mm, F.Cu at (65.2, 31.5)
- added D2: 1N4007, Diode_THT:D_DO-41_SOD81_P10.16mm_Horizontal, F.Cu at (215.0, 40.4)
- added D3: 1N4007, Diode_THT:D_DO-41_SOD81_P10.16mm_Horizontal, F.Cu at (215.0, 57.3)
- added D32: LED, LED_THT:LED_D5.0mm, F.Cu at (115.7, 144.0)
- added D33: LED, LED_THT:LED_D5.0mm, F.Cu at (123.7, 144.5)
- added D34: LED, LED_THT:LED_D5.0mm, F.Cu at (132.5, 144.5)
- added D35: LED, LED_THT:LED_D5.0mm, F.Cu at (140.2, 144.0)
- added D36: LED, LED_THT:LED_D5.0mm, F.Cu at (148.7, 144.0)
- added D37: LED, LED_THT:LED_D5.0mm, F.Cu at (156.7, 144.0)
- added D38: LED, LED_THT:LED_D5.0mm, F.Cu at (165.0, 144.0)
- added D39: LED, LED_THT:LED_D5.0mm, F.Cu at (173.0, 144.0)
- added D4: 1N4007, Diode_THT:D_DO-41_SOD81_P10.16mm_Horizontal, F.Cu at (215.0, 73.9)
- added D40: LED, LED_THT:LED_D5.0mm, F.Cu at (199.0, 39.5)
- added D41: LED, LED_THT:LED_D5.0mm, F.Cu at (199.0, 56.0)
- added D42: LED, LED_THT:LED_D5.0mm, F.Cu at (198.5, 73.0)
- added D43: LED, LED_THT:LED_D5.0mm, F.Cu at (199.0, 90.0)
- added D44: LED, LED_THT:LED_D5.0mm, F.Cu at (199.5, 108.0)
- added D45: LED, LED_THT:LED_D5.0mm, F.Cu at (197.5, 124.5)
- added D46: LED, LED_THT:LED_D5.0mm, F.Cu at (198.5, 141.5)
- added D47: LED, LED_THT:LED_D5.0mm, F.Cu at (198.0, 159.5)
- added D5: LED, LED_THT:LED_D5.0mm, F.Cu at (93.0, 109.5)
- added D6: 1N4007, Diode_THT:D_DO-41_SOD81_P10.16mm_Horizontal, F.Cu at (215.0, 91.4)
- added D7: 1N4007, Diode_THT:D_DO-41_SOD81_P10.16mm_Horizontal, F.Cu at (215.0, 108.3)
- added D8: 1N4007, Diode_THT:D_DO-41_SOD81_P10.16mm_Horizontal, F.Cu at (215.0, 125.4)
- added D9: 1N4007, Diode_THT:D_DO-41_SOD81_P10.16mm_Horizontal, F.Cu at (215.0, 142.5)
- added J1: Rookmachine, TerminalBlock_Phoenix:TerminalBlock_Phoenix_MKDS-1,5-2-5.08_1x02_P5.08mm_Horizontal, F.Cu at (117.9, 113.0)
- added J12: I/O nano, TerminalBlock_Phoenix:TerminalBlock_Phoenix_MKDS-1,5-4-5.08_1x04_P5.08mm_Horizontal, F.Cu at (77.5, 123.5)
- added J15: Relais 7&8, TerminalBlock_Phoenix:TerminalBlock_Phoenix_MKDS-1,5-4-5.08_1x04_P5.08mm_Horizontal, F.Cu at (247.5, 29.5)
- added J16: Alalog i/o, TerminalBlock_Phoenix:TerminalBlock_Phoenix_MKDS-1,5-5-5.08_1x05_P5.08mm_Horizontal, F.Cu at (137.0, 69.8)
- added J17: Extra 1-4, TerminalBlock_Phoenix:TerminalBlock_Phoenix_MKDS-1,5-4-5.08_1x04_P5.08mm_Horizontal, F.Cu at (151.0, 36.0)
- added J18: Extra 5-8, TerminalBlock_Phoenix:TerminalBlock_Phoenix_MKDS-1,5-4-5.08_1x04_P5.08mm_Horizontal, F.Cu at (172.3, 111.5)
- added J19: Relais 5&6, TerminalBlock_Phoenix:TerminalBlock_Phoenix_MKDS-1,5-4-5.08_1x04_P5.08mm_Horizontal, F.Cu at (247.5, 65.5)
- added J20: Relais 3&4, TerminalBlock_Phoenix:TerminalBlock_Phoenix_MKDS-1,5-4-5.08_1x04_P5.08mm_Horizontal, F.Cu at (247.3, 102.4)
- added J21: Relais 1&2, TerminalBlock_Phoenix:TerminalBlock_Phoenix_MKDS-1,5-4-5.08_1x04_P5.08mm_Horizontal, F.Cu at (247.0, 140.0)
- added J3: Power, TerminalBlock_Phoenix:TerminalBlock_Phoenix_MKDS-1,5-2-5.08_1x02_P5.08mm_Horizontal, F.Cu at (102.5, 113.2)
- added K10: SANYOU_SRD_Form_C, Relay_THT:Relay_SPDT_SANYOU_SRD_Series_Form_C, F.Cu at (219.8, 146.5)
- added K3: SANYOU_SRD_Form_C, Relay_THT:Relay_SPDT_SANYOU_SRD_Series_Form_C, F.Cu at (219.8, 27.5)
- added K4: SANYOU_SRD_Form_C, Relay_THT:Relay_SPDT_SANYOU_SRD_Series_Form_C, F.Cu at (219.8, 44.5)
- added K5: SANYOU_SRD_Form_C, Relay_THT:Relay_SPDT_SANYOU_SRD_Series_Form_C, F.Cu at (219.8, 61.5)
- added K6: SANYOU_SRD_Form_C, Relay_THT:Relay_SPDT_SANYOU_SRD_Series_Form_C, F.Cu at (219.8, 78.5)
- added K7: SANYOU_SRD_Form_C, Relay_THT:Relay_SPDT_SANYOU_SRD_Series_Form_C, F.Cu at (219.8, 95.5)
- added K8: SANYOU_SRD_Form_C, Relay_THT:Relay_SPDT_SANYOU_SRD_Series_Form_C, F.Cu at (219.8, 112.5)
- added K9: SANYOU_SRD_Form_C, Relay_THT:Relay_SPDT_SANYOU_SRD_Series_Form_C, F.Cu at (219.8, 129.5)
- added Q1: BC547, Package_TO_SOT_THT:TO-92_Inline, F.Cu at (119.2, 101.4)
- added Q10: BC337, Package_TO_SOT_THT:TO-92_Inline, F.Cu at (209.5, 84.0)
- added Q11: BC337, Package_TO_SOT_THT:TO-92_Inline, F.Cu at (209.5, 101.5)
- added Q12: BC337, Package_TO_SOT_THT:TO-92_Inline, F.Cu at (209.5, 118.5)
- added Q13: BC337, Package_TO_SOT_THT:TO-92_Inline, F.Cu at (209.5, 136.0)
- added Q14: BC337, Package_TO_SOT_THT:TO-92_Inline, F.Cu at (209.5, 152.5)
- added Q4: Q_NMOS_GSD, PCM_SparkFun-Semiconductor-Standard:SC-89 SOT-490, F.Cu at (80.7, 55.9)
- added Q5: BC337, Package_TO_SOT_THT:TO-92_Inline, F.Cu at (209.5, 33.5)
- added Q6: BC337, Package_TO_SOT_THT:TO-92_Inline, F.Cu at (209.5, 50.5)
- added Q7: Q_NMOS_GSD, PCM_SparkFun-Semiconductor-Standard:SC-89 SOT-490, F.Cu at (76.7, 45.1)
- added Q8: Q_NMOS_GSD, PCM_SparkFun-Semiconductor-Standard:SC-89 SOT-490, F.Cu at (76.2, 37.9)
- added Q9: BC337, Package_TO_SOT_THT:TO-92_Inline, F.Cu at (209.5, 67.5)
- added R14: 1K, Resistor_THT:R_Axial_DIN0204_L3.6mm_D1.6mm_P7.62mm_Horizontal, F.Cu at (83.9, 83.5)
- added R15: 1K, Resistor_THT:R_Axial_DIN0204_L3.6mm_D1.6mm_P7.62mm_Horizontal, F.Cu at (84.4, 78.0)
- added R16: 1K, Resistor_THT:R_Axial_DIN0204_L3.6mm_D1.6mm_P7.62mm_Horizontal, F.Cu at (82.9, 73.5)
- added R23: 120R, Resistor_THT:R_Axial_DIN0204_L3.6mm_D1.6mm_P7.62mm_Horizontal, F.Cu at (95.5, 60.5)
- added R24: 10K, Resistor_THT:R_Axial_DIN0204_L3.6mm_D1.6mm_P7.62mm_Horizontal, F.Cu at (87.4, 56.0)
- added R25: 1K, Resistor_THT:R_Axial_DIN0204_L3.6mm_D1.6mm_P7.62mm_Horizontal, F.Cu at (59.6, 57.5)
- added R26: 120R, Resistor_THT:R_Axial_DIN0204_L3.6mm_D1.6mm_P7.62mm_Horizontal, F.Cu at (87.4, 48.0)
- added R27: 10K, Resistor_THT:R_Axial_DIN0204_L3.6mm_D1.6mm_P7.62mm_Horizontal, F.Cu at (86.9, 42.5)
- added R28: 1K, Resistor_THT:R_Axial_DIN0204_L3.6mm_D1.6mm_P7.62mm_Horizontal, F.Cu at (53.4, 39.5)
- added R29: 120R, Resistor_THT:R_Axial_DIN0204_L3.6mm_D1.6mm_P7.62mm_Horizontal, F.Cu at (90.4, 26.0)
- added R30: 10K, Resistor_THT:R_Axial_DIN0204_L3.6mm_D1.6mm_P7.62mm_Horizontal, F.Cu at (90.7, 18.0)
- added R31: 1K, Resistor_THT:R_Axial_DIN0204_L3.6mm_D1.6mm_P7.62mm_Horizontal, F.Cu at (64.4, 22.0)
- added R34: 680, Resistor_THT:R_Axial_DIN0204_L3.6mm_D1.6mm_P7.62mm_Horizontal, F.Cu at (198.2, 30.0)
- added R35: 680, Resistor_THT:R_Axial_DIN0204_L3.6mm_D1.6mm_P7.62mm_Horizontal, F.Cu at (198.2, 46.0)
- added R36: 680, Resistor_THT:R_Axial_DIN0204_L3.6mm_D1.6mm_P7.62mm_Horizontal, F.Cu at (198.2, 63.0)
- added R37: 680, Resistor_THT:R_Axial_DIN0204_L3.6mm_D1.6mm_P7.62mm_Horizontal, F.Cu at (197.7, 79.5)
- added R38: 680, Resistor_THT:R_Axial_DIN0204_L3.6mm_D1.6mm_P7.62mm_Horizontal, F.Cu at (197.2, 97.5)
- added R39: 680, Resistor_THT:R_Axial_DIN0204_L3.6mm_D1.6mm_P7.62mm_Horizontal, F.Cu at (196.7, 114.5)
- added R40: 680, Resistor_THT:R_Axial_DIN0204_L3.6mm_D1.6mm_P7.62mm_Horizontal, F.Cu at (196.2, 131.5)
- added R41: 680, Resistor_THT:R_Axial_DIN0204_L3.6mm_D1.6mm_P7.62mm_Horizontal, F.Cu at (195.2, 147.5)
- added R44: 1K, Resistor_THT:R_Axial_DIN0204_L3.6mm_D1.6mm_P7.62mm_Horizontal, F.Cu at (163.1, 61.0)
- added R45: 1K, Resistor_THT:R_Axial_DIN0204_L3.6mm_D1.6mm_P7.62mm_Horizontal, F.Cu at (155.5, 63.5)
- added R46: 1K, Resistor_THT:R_Axial_DIN0204_L3.6mm_D1.6mm_P7.62mm_Horizontal, F.Cu at (155.5, 66.5)
- added R47: 1K, Resistor_THT:R_Axial_DIN0204_L3.6mm_D1.6mm_P7.62mm_Horizontal, F.Cu at (155.7, 68.5)
- added R48: 1K, Resistor_THT:R_Axial_DIN0204_L3.6mm_D1.6mm_P7.62mm_Horizontal, F.Cu at (155.8, 71.0)
- added R49: 1K, Resistor_THT:R_Axial_DIN0204_L3.6mm_D1.6mm_P7.62mm_Horizontal, F.Cu at (155.7, 73.5)
- added R50: 1K, Resistor_THT:R_Axial_DIN0204_L3.6mm_D1.6mm_P7.62mm_Horizontal, F.Cu at (155.5, 76.0)
- added R51: 1K, Resistor_THT:R_Axial_DIN0204_L3.6mm_D1.6mm_P7.62mm_Horizontal, F.Cu at (155.5, 79.0)
- added R52: 1K, Resistor_THT:R_Axial_DIN0204_L3.6mm_D1.6mm_P7.62mm_Horizontal, F.Cu at (198.2, 34.0)
- added R53: 1K, Resistor_THT:R_Axial_DIN0204_L3.6mm_D1.6mm_P7.62mm_Horizontal, F.Cu at (198.2, 50.5)
- added R54: 1K, Resistor_THT:R_Axial_DIN0204_L3.6mm_D1.6mm_P7.62mm_Horizontal, F.Cu at (198.2, 67.5)
- added R55: 1K, Resistor_THT:R_Axial_DIN0204_L3.6mm_D1.6mm_P7.62mm_Horizontal, F.Cu at (197.7, 84.0)
- added R56: 1K, Resistor_THT:R_Axial_DIN0204_L3.6mm_D1.6mm_P7.62mm_Horizontal, F.Cu at (197.2, 101.5)
- added R57: 1K, Resistor_THT:R_Axial_DIN0204_L3.6mm_D1.6mm_P7.62mm_Horizontal, F.Cu at (196.7, 119.0)
- added R58: 1K, Resistor_THT:R_Axial_DIN0204_L3.6mm_D1.6mm_P7.62mm_Horizontal, F.Cu at (196.2, 136.0)
- added R59: 1K, Resistor_THT:R_Axial_DIN0204_L3.6mm_D1.6mm_P7.62mm_Horizontal, F.Cu at (195.2, 152.5)
- added R7: 1500, Resistor_THT:R_Axial_DIN0204_L3.6mm_D1.6mm_P7.62mm_Horizontal, F.Cu at (106.2, 97.5)
- added R8: 10k, Resistor_THT:R_Axial_DIN0204_L3.6mm_D1.6mm_P7.62mm_Horizontal, F.Cu at (181.3, 36.0)
- added R9: 1K, Resistor_THT:R_Axial_DIN0204_L3.6mm_D1.6mm_P7.62mm_Horizontal, F.Cu at (93.2, 97.5)
- moved U1 43.1 mm to (181.3, 78.0), turned to 180 degrees
- moved A1 26.6 mm to (105.8, 48.0)
Connections:
- net Earth renamed GND
- net Net-(A1-3V3) renamed +3.3V
- A1 pad 10: unconnected-(A1-D7-Pad10) -> Net-(A1-D7)
- A1 pad 11: unconnected-(A1-D8-Pad11) -> Net-(A1-D8)
- A1 pad 12: unconnected-(A1-D9-Pad12) -> Net-(A1-D9)
- A1 pad 19: unconnected-(A1-A0-Pad19) -> Net-(A1-A0)
- A1 pad 20: unconnected-(A1-A1-Pad20) -> Net-(A1-A1)
- A1 pad 21: unconnected-(A1-A2-Pad21) -> Net-(A1-A2)
- A1 pad 22: unconnected-(A1-A3-Pad22) -> Net-(A1-A3)
- A1 pad 25: unconnected-(A1-A6-Pad25) -> Net-(A1-A6)
- A1 pad 26: unconnected-(A1-A7-Pad26) -> Net-(A1-A7)
- A1 pad 5: unconnected-(A1-D2-Pad5) -> Net-(A1-D2)
- A1 pad 6: unconnected-(A1-D3-Pad6) -> Net-(A1-D3)
- A1 pad 7: unconnected-(A1-D4-Pad7) -> Net-(A1-D4)
- A1 pad 8: unconnected-(A1-D5-Pad8) -> Net-(A1-D5)
- A1 pad 9: unconnected-(A1-D6-Pad9) -> Net-(A1-D6)
- U1 pad 1: unconnected-(U1-GPB0-Pad1) -> Net-(U1-GPB0)
- U1 pad 2: unconnected-(U1-GPB1-Pad2) -> Net-(U1-GPB1)
- U1 pad 21: unconnected-(U1-GPA0-Pad21) -> Net-(J17-Pin_1)
- U1 pad 22: unconnected-(U1-GPA1-Pad22) -> Net-(J17-Pin_2)
- U1 pad 23: unconnected-(U1-GPA2-Pad23) -> Net-(J17-Pin_3)
- U1 pad 24: unconnected-(U1-GPA3-Pad24) -> Net-(J17-Pin_4)
- U1 pad 25: unconnected-(U1-GPA4-Pad25) -> Net-(J18-Pin_1)
- U1 pad 26: unconnected-(U1-GPA5-Pad26) -> Net-(J18-Pin_2)
- U1 pad 27: unconnected-(U1-GPA6-Pad27) -> Net-(J18-Pin_3)
- U1 pad 28: unconnected-(U1-GPA7-Pad28) -> Net-(J18-Pin_4)
- U1 pad 3: unconnected-(U1-GPB2-Pad3) -> Net-(U1-GPB2)
- U1 pad 4: unconnected-(U1-GPB3-Pad4) -> Net-(U1-GPB3)
- U1 pad 5: unconnected-(U1-GPB4-Pad5) -> Net-(U1-GPB4)
- U1 pad 6: unconnected-(U1-GPB5-Pad6) -> Net-(U1-GPB5)
- U1 pad 7: unconnected-(U1-GPB6-Pad7) -> Net-(U1-GPB6)
- U1 pad 8: unconnected-(U1-GPB7-Pad8) -> Net-(U1-GPB7)

Commit message: pcb update
Parts:
- removed D10, D11, D12, D15, D16: LED, LED_THT:LED_D5.0mm
- removed Q4, Q7, Q8: Q_NMOS_GSD, PCM_SparkFun-Semiconductor-Standard:SC-89 SOT-490
- removed R14, R15, R16, R25, R28: 1K, Resistor_THT:R_Axial_DIN0204_L3.6mm_D1.6mm_P7.62mm_Horizontal
- added Q15: IRLZ44N, Package_TO_SOT_THT:TO-220-3_Vertical, F.Cu at (68.9, 32.0)
- added Q2: IRLZ44N, Package_TO_SOT_THT:TO-220-3_Vertical, F.Cu at (65.4, 69.5)
- added Q3: IRLZ44N, Package_TO_SOT_THT:TO-220-3_Vertical, F.Cu at (68.9, 50.5)
- added R61: 4k7, Resistor_THT:R_Axial_DIN0204_L3.6mm_D1.6mm_P7.62mm_Horizontal, F.Cu at (127.5, 71.8)
- added R62: 4k7, Resistor_THT:R_Axial_DIN0204_L3.6mm_D1.6mm_P7.62mm_Horizontal, F.Cu at (134.0, 72.8)
- Q1: value BC547 -> BC337
- moved R31 128.3 mm to (53.0, 149.8), turned to 90 degrees
- moved D17 115.5 mm to (44.0, 145.0)
- moved R44 100.8 mm to (112.5, 148.1), turned to 90 degrees
- moved R45 91.5 mm to (119.8, 147.7), turned to 90 degrees
- moved R46 86.7 mm to (127.0, 148.4), turned to 90 degrees
- moved R47 82.3 mm to (134.0, 147.9), turned to 90 degrees
- moved R48 78.5 mm to (142.0, 148.2), turned to 90 degrees
- moved R49 74.5 mm to (149.8, 147.7), turned to 90 degrees
- moved J3 73.6 mm to (46.0, 160.5)
- moved R50 72.1 mm to (156.8, 148.1), turned to 90 degrees
- moved R51 69.2 mm to (163.5, 147.7), turned to 90 degrees
- moved D39 61.6 mm to (112.5, 155.6)
- moved R30 51.6 mm to (65.5, 63.0)
- moved R29 51.5 mm to (73.0, 74.5), turned to 180 degrees
- moved D32 48.6 mm to (163.2, 154.4)
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Connections:
- D17 pad 1: Net-(D17-K) -> GND
- U1 pad 15: unconnected-(U1-A0-Pad15) -> GND
- U1 pad 16: unconnected-(U1-A1-Pad16) -> GND
- U1 pad 17: unconnected-(U1-A2-Pad17) -> GND
Routing:
- net GND: track 0.00 -> 1623.5 mm
- net +5V: track 0.00 -> 755.8 mm
- net +3.3V: track 0.00 -> 399.7 mm
- net Net-(J17-Pin_1): track 0.00 -> 110.0 mm
- net Net-(J17-Pin_2): track 0.00 -> 102.5 mm
- net Net-(A1-SDA/A4): track 0.00 -> 96.8 mm
- net Net-(J17-Pin_3): track 0.00 -> 96.2 mm
- net Net-(J18-Pin_1): track 0.00 -> 89.5 mm
- net Net-(A1-A0): track 0.00 -> 89.2 mm
- net Net-(J17-Pin_4): track 0.00 -> 88.9 mm
- net Net-(J18-Pin_2): track 0.00 -> 86.5 mm
- net Net-(J18-Pin_3): track 0.00 -> 83.5 mm
- net Net-(J18-Pin_4): track 0.00 -> 81.5 mm
- net Net-(U1-GPB0): track 0.00 -> 81.4 mm
- net Net-(A1-SCL/A5): track 0.00 -> 76.1 mm
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