File: schakelbord/schakelbord/schakelbord.kicad_pcb (KiCad board)
At the start: 2 copper layers, 200 x 170 mm, 111 parts, among them J1 Screw_Terminal_01x03, J12 I/O nano, J15 Relais 7&8, J16 Alalog i/o, J17 Extra 1-4, J18 Extra 5-8, J19 Relais 5&6, J20 Relais 3&4, J21 Relais 1&2, J3 Power, J4 mosfets, K10 SANYOU_SRD_Form_C, K3 SANYOU_SRD_Form_C, K4 SANYOU_SRD_Form_C, K5 SANYOU_SRD_Form_C, K6 SANYOU_SRD_Form_C, K7 SANYOU_SRD_Form_C, K8 SANYOU_SRD_Form_C, K9 SANYOU_SRD_Form_C, Q1 BC337, Q10 BC337, Q11 BC337, Q12 BC337, Q13 BC337, Q14 BC337, Q15 IRLZ44N, Q2 IRLZ44N, Q3 IRLZ44N, Q5 BC337, Q6 BC337, Q9 BC337, U1 MCP23017x-x-SP

Commit message: pcb update
Parts:
- added C1: 0.1uF, Capacitor_THT:C_Disc_D3.0mm_W1.6mm_P2.50mm, F.Cu at (153.2, 118.2)
- added C2: 470uF, PCM_SparkFun-Capacitor:Electrolytic_10.3x10.3mm, F.Cu at (87.8, 86.0)
Connections:
- D32 pad 2: +5V -> +3.3V
- D33 pad 2: +5V -> +3.3V
- D34 pad 2: +5V -> +3.3V
- D35 pad 2: +5V -> +3.3V
- D36 pad 2: +5V -> +3.3V
- D37 pad 2: +5V -> +3.3V
- D38 pad 2: +5V -> +3.3V
- D39 pad 2: +5V -> +3.3V
- D49 pad 2: +5V -> +3.3V
- D50 pad 2: +5V -> +3.3V
- D51 pad 2: +5V -> +3.3V
- D52 pad 2: +5V -> +3.3V
- D53 pad 1: Net-(D53-K) -> GND
- D53 pad 2: +5V -> Net-(D53-A)
- D54 pad 1: Net-(D54-K) -> GND
- D54 pad 2: +5V -> Net-(D54-A)
- D55 pad 1: Net-(D55-K) -> GND
- D55 pad 2: +5V -> Net-(D55-A)
- R67 pad 1: Net-(D53-K) -> Net-(A1-D2)
- R67 pad 2: Net-(A1-D4) -> Net-(D53-A)
- R68 pad 1: Net-(D54-K) -> Net-(A1-D3)
- R68 pad 2: Net-(A1-D3) -> Net-(D54-A)
- R69 pad 1: Net-(D55-K) -> Net-(A1-D4)
- R69 pad 2: Net-(A1-D2) -> Net-(D55-A)
Routing:
- net +5V: track 829.1 -> 702.8 mm
- net +3.3V: track 166.0 -> 281.8 mm
- net Net-(D55-K): track 19.8 -> 0.00 mm
- net Net-(D53-K): track 19.1 -> 0.00 mm
- net Net-(D54-K): track 19.0 -> 0.00 mm
- net (no net): track 0.00 -> 19.0 mm
- net GND: track 1184.3 -> 1192.6 mm

Commit message: pcb update
Parts:
- removed D49, D50, D51, D52: LED, LED_THT:LED_D5.0mm
- removed J12: I/O nano, TerminalBlock_Phoenix:TerminalBlock_Phoenix_MKDS-1,5-4-5.08_1x04_P5.08mm_Horizontal
- removed R63, R64, R65, R66: 1K, Resistor_THT:R_Axial_DIN0204_L3.6mm_D1.6mm_P7.62mm_Horizontal
- added J22: Input pins, TerminalBlock_Phoenix:TerminalBlock_Phoenix_MKDS-1,5-5-5.08_1x05_P5.08mm_Horizontal, F.Cu at (72.2, 135.8)
- moved D55 45.9 mm to (81.5, 75.2)
- moved R67 44.6 mm to (96.3, 33.2), turned to 180 degrees
- moved D53 43.0 mm to (81.5, 34.2)
- moved R69 38.9 mm to (96.3, 75.5), turned to 180 degrees
- moved R30 16.0 mm to (88.7, 78.8)
- moved R27 13.0 mm to (88.7, 58.2)
- moved J4 12.5 mm to (72.2, 65.2)
- moved R24 12.3 mm to (88.7, 36.8)
- moved D54 12.1 mm to (81.5, 55.8)
- moved R68 8.60 mm to (96.5, 54.2), turned to 180 degrees
- moved Q15 5.08 mm to (88.7, 25.7)
- moved R23 5.02 mm to (96.3, 29.8)
- moved D17 4.50 mm to (66.5, 145.2)
- moved Q3 4.28 mm to (88.7, 46.0)
- moved R26 4.08 mm to (96.3, 50.2)
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Routing:
- net +3.3V: track 281.8 -> 332.7 mm
- net Net-(A1-D5): track 141.0 -> 92.0 mm
- net Net-(A1-D6): track 135.6 -> 93.6 mm
- net GND: track 1192.6 -> 1227.3 mm, vias 4 -> 2
- net Net-(J4-Pin_3): track 26.5 -> 52.8 mm
- net Net-(J1-Pin_3): track 68.7 -> 94.1 mm, vias 2 -> 0
- net Net-(A1-D8): track 117.2 -> 96.3 mm
- net Net-(A1-D7): track 114.3 -> 95.1 mm
- net (no net): track 19.0 -> 0.00 mm
- net Net-(J4-Pin_2): track 26.8 -> 36.7 mm
- net Net-(A1-D9): track 66.5 -> 57.2 mm
- net Net-(D51-K): track 7.76 -> 0.00 mm
- net Net-(D50-K): track 7.71 -> 0.00 mm
- net Net-(D49-K): track 7.71 -> 0.00 mm
- net Net-(D52-K): track 7.65 -> 0.00 mm
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
Commit message: pcb update
Parts:
- A1, D1, D17, D2, D3, D32, D33, D34, D35, D36, D37, D38, D39, D4, D40, D41, D42, D43, D44, D45, D46, D47, D5, D53, D54, D55, D6, D7, D8, D9, J1, J15, J16, J17, J18, J19, J20, J21, J22, J3, J4, K10, K3, K4, K5, K6, K7, K8, K9, Q15, Q2, Q3, R1, R2, R23, R24, R26, R27, R29, R30, R31, R34, R35, R36, R37, R38, R39, R40, R41, R44, R45, R46, R47, R48, R49, R50, R51, R52, R53, R54, R55, R56, R57, R58, R59, R61, R62, R67, R68, R69, R7, R8, R9, U1: moved to B.Cu
- C1: footprint Capacitor_THT:C_Disc_D3.0mm_W1.6mm_P2.50mm -> Capacitor_THT:C_Disc_D5.0mm_W2.5mm_P5.00mm; moved to B.Cu
- C2: footprint PCM_SparkFun-Capacitor:Electrolytic_10.3x10.3mm -> Capacitor_THT:CP_Radial_D8.0mm_P3.50mm; moved to B.Cu
- Q1, Q10, Q11, Q12, Q13, Q14, Q5, Q6, Q9: footprint Package_TO_SOT_THT:TO-92_Inline -> Package_TO_SOT_THT:TO-92L_Inline_Wide; moved to B.Cu
- moved J21 184.0 mm to (64.0, 148.7)
- moved J15 183.0 mm to (64.5, 42.7)
- moved J19 183.0 mm to (64.5, 77.7)
- moved J20 183.0 mm to (64.5, 113.7)
- moved D17 179.1 mm to (245.5, 145.2), turned to 180 degrees
- moved J3 176.5 mm to (244.2, 158.2), turned to 180 degrees
- moved J1 167.5 mm to (239.8, 107.7)
- moved J22 167.5 mm to (239.8, 135.8)
- moved J4 167.5 mm to (239.8, 65.2)
- moved R31 161.5 mm to (236.8, 149.3)
- moved D53 149.1 mm to (230.5, 34.2), turned to 180 degrees
- moved D54 149.1 mm to (230.5, 55.8), turned to 180 degrees
- moved D55 149.1 mm to (230.5, 75.2), turned to 180 degrees
- moved C2 140.5 mm to (228.2, 86.0), turned to 180 degrees
- moved R24 134.6 mm to (223.3, 36.8), turned to 180 degrees
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Routing:
- net Net-(A1-A7): track 83.6 -> 74.3 mm
- net Net-(J17-Pin_1): track 191.9 -> 200.4 mm
- net Net-(A1-SCL/A5): track 123.1 -> 131.6 mm
- net Net-(J17-Pin_2): track 186.3 -> 192.6 mm
- net Net-(A1-D4): track 41.7 -> 35.7 mm
- net Net-(A1-D2): track 60.4 -> 54.4 mm
- net Net-(A1-D3): track 48.7 -> 42.7 mm
- net Net-(A1-A0): track 121.4 -> 127.1 mm
- net Net-(J17-Pin_3): track 175.7 -> 180.8 mm
- net Net-(A1-SDA/A4): track 133.9 -> 138.3 mm
- net Net-(A1-D5): track 92.0 -> 87.7 mm
- net +3.3V: track 332.7 -> 329.0 mm
- net Net-(J18-Pin_2): track 138.3 -> 141.7 mm
- net Net-(J18-Pin_3): track 126.7 -> 130.1 mm
- net Net-(A1-A6): track 59.0 -> 55.8 mm
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Other:
- board size 200 x 170 mm -> 197.5 x 161 mm
