File: schakelbord/schakelbord/schakelbord-first.kicad_pcb (KiCad board)
At the start: 2 copper layers, 200 x 170 mm, 111 parts, among them J1 Screw_Terminal_01x03, J12 I/O nano, J15 Relais 7&8, J16 Alalog i/o, J17 Extra 1-4, J18 Extra 5-8, J19 Relais 5&6, J20 Relais 3&4, J21 Relais 1&2, J3 Power, J4 mosfets, K10 SANYOU_SRD_Form_C, K3 SANYOU_SRD_Form_C, K4 SANYOU_SRD_Form_C, K5 SANYOU_SRD_Form_C, K6 SANYOU_SRD_Form_C, K7 SANYOU_SRD_Form_C, K8 SANYOU_SRD_Form_C, K9 SANYOU_SRD_Form_C, Q1 BC337, Q10 BC337, Q11 BC337, Q12 BC337, Q13 BC337, Q14 BC337, Q15 IRLZ44N, Q2 IRLZ44N, Q3 IRLZ44N, Q5 BC337, Q6 BC337, Q9 BC337, U1 MCP23017x-x-SP

Commit message: pcb update
Parts:
- R9: footprint Resistor_THT:R_Axial_DIN0207_L6.3mm_D2.5mm_P10.16mm_Horizontal -> Resistor_THT:R_Axial_DIN0204_L3.6mm_D1.6mm_P7.62mm_Horizontal
- moved J17 62.2 mm to (147.5, 78.9), turned to -90 degrees
- moved J18 60.7 mm to (147.5, 103.0), turned to -90 degrees
- moved J1 45.5 mm to (117.5, 112.0), turned to 0 degrees
- moved J16 44.8 mm to (145.0, 68.3), turned to 90 degrees
- moved R61 44.0 mm to (127.5, 71.8)
- moved Q1 43.5 mm to (130.0, 76.5)
- moved R62 43.0 mm to (134.0, 72.8)
- moved R2 35.0 mm to (97.3, 98.0)
- moved R9 30.5 mm to (89.2, 82.5)
- moved A1 30.4 mm to (105.8, 48.0)
- moved R7 30.0 mm to (110.2, 96.0)
- moved R1 29.7 mm to (119.3, 100.0), turned to 180 degrees
- moved D53 27.7 mm to (47.3, 77.5), turned to 180 degrees
- moved D5 27.3 mm to (77.5, 83.0)
- moved J12 26.1 mm to (47.0, 124.0)
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Routing:
- net GND: track 1184.3 -> 1389.9 mm, vias 4 -> 2
- net +5V: track 829.1 -> 1005.1 mm, vias 0 -> 2
- net Net-(J17-Pin_2): track 186.3 -> 102.5 mm, vias 2 -> 0
- net Net-(J17-Pin_4): track 170.9 -> 88.9 mm, vias 2 -> 0
- net Net-(J17-Pin_1): track 191.7 -> 110.0 mm, vias 2 -> 0
- net Net-(J17-Pin_3): track 174.8 -> 96.2 mm, vias 2 -> 0
- net +3.3V: track 166.0 -> 228.9 mm
- net Net-(J18-Pin_1): track 150.7 -> 89.5 mm
- net Net-(A1-A1): track 79.3 -> 26.1 mm, vias 2 -> 0
- net Net-(J18-Pin_2): track 138.3 -> 86.5 mm
- net Net-(J1-Pin_3): track 68.7 -> 17.0 mm, vias 2 -> 0
- net Net-(A1-A2): track 77.5 -> 27.2 mm, vias 2 -> 0
- net Net-(A1-A3): track 76.6 -> 28.2 mm, vias 2 -> 0
- net Net-(A1-SCL/A5): track 123.1 -> 78.9 mm
- net Net-(J18-Pin_3): track 126.7 -> 83.5 mm
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Other:
- board outline removed
