File: schakelbord/schakelbord/schakelbord.kicad_sch (KiCad schematic)
At the start: 113 parts, among them J1 Power, J10 Relais 5&6, J11 Relais 1&2, J2 Generic output, J3 Mosfets, J4 Analog input, J5 Fogger, J6 Extra 1-4, J7 Extra 5-8, J8 Relais 7&8, J9 Relais 3&4, K1 SANYOU_SRD_Form_C, K2 SANYOU_SRD_Form_C, K3 SANYOU_SRD_Form_C, K4 SANYOU_SRD_Form_C, K5 SANYOU_SRD_Form_C, K6 SANYOU_SRD_Form_C, K7 SANYOU_SRD_Form_C, K8 SANYOU_SRD_Form_C, Q1 IRLZ44N, Q10 BC337, Q11 BC337, Q12 BC337, Q2 IRLZ44N, Q3 IRLZ44N, Q4 BC337, Q5 BC337, Q6 BC337, Q7 BC337, Q8 BC337, Q9 BC337, U1 MCP23017

Commit message: Revert "Cleanup"
This reverts commit 4277aa74836c99404227eb422add9ba860ad75b2.
Parts:
- removed D10, D11, D12, D13, D14, D15, D16, D17, D2, D4, D5, D6, D7, D8: LED, LED_THT:LED_D5.0mm, symbol Device:LED
- removed R1, R11, R12, R13, R14, R2, R22, R23, R24, R25, R26, R27, R28, R29, R4: 470, symbol Device:R
- removed R17, R20: 4k7, symbol Device:R
- added D32, D33, D34, D35, D36, D37, D38, D39, D49, D50, D51, D52, D54, D55: LED, LED_THT:LED_D5.0mm, symbol Device:LED
- added R44, R45, R46, R47, R48, R49, R50, R51, R63, R64, R65, R66, R67, R68, R69: 1K, Resistor_THT:R_Axial_DIN0204_L3.6mm_D1.6mm_P7.62mm_Horizontal, symbol Device:R
- added R61, R62: 4k7, Resistor_THT:R_Axial_DIN0204_L3.6mm_D1.6mm_P7.62mm_Horizontal, symbol Device:R
- J1: renamed from J5; value Fogger -> Screw_Terminal_01x03
- J12: renamed from J2; value Generic output -> I/O nano
- J16: renamed from J4; value Analog input -> Alalog i/o
- J4: renamed from J3; value Mosfets -> mosfets
- R9: renamed from R15; value 470 -> 1K
- U1: value MCP23017 -> MCP23017x-x-SP
- renumbered C2 to C1, C1 to C2, D22 to D1, D3 to D17, D30 to D2, D24 to D3, D32 to D4, D18 to D40, D26 to D41, D20 to D42, D28 to D43, D19 to D44, D27 to D45, D21 to D46, D29 to D47, D9 to D5, D1 to D53, D23 to D6, D31 to D7, D25 to D8, D33 to D9, J8 to J15, J6 to J17, J7 to J18, J10 to J19, J9 to J20, J11 to J21, J1 to J3, K8 to K10, K1 to K3, K5 to K4, K3 to K5, K7 to K6, K2 to K7, K6 to K8, K4 to K9, Q4 to Q1, Q11 to Q10, Q6 to Q11, Q10 to Q12, Q8 to Q13, Q12 to Q14, Q2 to Q15, Q3 to Q2, Q1 to Q3, Q9 to Q6, Q7 to Q9, R18 to R1, R19 to R2, R7 to R23, R9 to R24, R6 to R26, R8 to R27, R5 to R29, R10 to R30, R3 to R31, R42 to R35, R44 to R37, R35 to R38, R43 to R39, R37 to R40, R45 to R41, R30 to R52, R38 to R53, R32 to R54, R40 to R55, R31 to R56, R39 to R57, R33 to R58, R41 to R59, R16 to R7, R21 to R8
Connections:
- net +3.3V: now also U1.9 (V_{DD}), D32.2 (A), D33.2 (A), D34.2 (A), D35.2 (A), D36.2 (A), D37.2 (A), D38.2 (A), D39.2 (A), D49.2 (A), D50.2 (A), D51.2 (A), D52.2 (A), R61.1, R62.1
- net GND: now also J16.5 (Pin_5), D54.1 (K), D55.1 (K); no longer J16.1 (Pin_1)
- net at J17.2 (Pin_2), U1.22 (GPA1): now also R45.2
- net at A1.6 (D3): now also R26.1, R68.1; no longer J12.3 (Pin_3)
- net at J18.1 (Pin_1), U1.25 (GPA4): now also R48.2
- net at J18.2 (Pin_2), U1.26 (GPA5): now also R49.2
- net at J18.3 (Pin_3), U1.27 (GPA6): now also R50.2
- net at J18.4 (Pin_4), U1.28 (GPA7): now also R51.2
- net at A1.11 (D8): now also J12.1 (Pin_1), R63.2; no longer R29.1
- net at D53.2 (A): now also R67.2
- net at A1.10 (D7): now also J12.2 (Pin_2), R64.2; no longer R26.1
- net at A1.19 (A0): now also J1.1 (Pin_1), Q1.1 (C); no longer J16.2 (Pin_2)
- net at A1.20 (A1): now also J16.1 (Pin_1); no longer J16.3 (Pin_3)
- net at A1.21 (A2): now also J16.2 (Pin_2); no longer J16.4 (Pin_4)
- net at A1.22 (A3): now also J16.3 (Pin_3); no longer J16.5 (Pin_5)
- net at A1.23 (SDA/A4), U1.13 (SDA): now also R62.2
- net at A1.24 (SCL/A5), U1.12 (SCK): now also R61.2
- net at A1.5 (D2): now also R23.1, R67.1; no longer J12.4 (Pin_4)
- net at A1.7 (D4): now also R29.1, R69.1; no longer J12.2 (Pin_2)
- net at A1.8 (D5): now also J12.4 (Pin_4), R66.2; no longer J12.1 (Pin_1)
- net at A1.9 (D6): now also J12.3 (Pin_3), R65.2; no longer R23.1
- net at J17.1 (Pin_1), U1.21 (GPA0): now also R44.2
- net at J17.3 (Pin_3), U1.23 (GPA2): now also R46.2
- net at J17.4 (Pin_4), U1.24 (GPA3): now also R47.2
- new net: D50.1 (K), R64.1
- new net: D55.2 (A), R69.2
- new net: D52.1 (K), R66.1
- new net: A1.25 (A6), J16.4 (Pin_4)
- new net: D54.2 (A), R68.2
- new net: D37.1 (K), R46.1
- new net: D34.1 (K), R49.1
- new net: D33.1 (K), R50.1
- new net: D39.1 (K), R44.1
- new net: D36.1 (K), R47.1
- new net: D35.1 (K), R48.1
- new net: D51.1 (K), R65.1
- new net: D32.1 (K), R51.1
- new net: D49.1 (K), R63.1
- new net: D38.1 (K), R45.1
Other:
- moved on the sheet: A1, C1, C2, D1, D17, D2, D3, D4, D40, D41, D42, D43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

Commit message: Cleanup
Parts:
- removed D32, D33, D34, D35, D36, D37, D38, D39, D49, D50, D51, D52, D54, D55: LED, LED_THT:LED_D5.0mm, symbol Device:LED
- removed R44, R45, R46, R47, R48, R49, R50, R51, R63, R64, R65, R66, R67, R68, R69: 1K, Resistor_THT:R_Axial_DIN0204_L3.6mm_D1.6mm_P7.62mm_Horizontal, symbol Device:R
- removed R61, R62: 4k7, Resistor_THT:R_Axial_DIN0204_L3.6mm_D1.6mm_P7.62mm_Horizontal, symbol Device:R
- added D10, D11, D12, D13, D14, D15, D16, D17, D2, D4, D5, D6, D7, D8: LED, LED_THT:LED_D5.0mm, symbol Device:LED
- added R1, R11, R12, R13, R14, R2, R22, R23, R24, R25, R26, R27, R28, R29, R4: 470, symbol Device:R
- added R17, R20: 4k7, symbol Device:R
- J2: renamed from J12; value I/O nano -> Generic output
- J3: renamed from J4; value mosfets -> Mosfets
- J4: renamed from J16; value Alalog i/o -> Analog input
- J5: renamed from J1; value Screw_Terminal_01x03 -> Fogger
- R15: renamed from R9; value 1K -> 470
- U1: value MCP23017x-x-SP -> MCP23017
- renumbered C2 to C1, C1 to C2, D53 to D1, D40 to D18, D44 to D19, D42 to D20, D46 to D21, D1 to D22, D6 to D23, D3 to D24, D8 to D25, D41 to D26, D45 to D27, D43 to D28, D47 to D29, D17 to D3, D2 to D30, D7 to D31, D4 to D32, D9 to D33, D5 to D9, J3 to J1, J19 to J10, J21 to J11, J17 to J6, J18 to J7, J15 to J8, J20 to J9, K3 to K1, K7 to K2, K5 to K3, K9 to K4, K4 to K5, K8 to K6, K6 to K7, K10 to K8, Q3 to Q1, Q12 to Q10, Q10 to Q11, Q14 to Q12, Q15 to Q2, Q2 to Q3, Q1 to Q4, Q11 to Q6, Q9 to Q7, Q13 to Q8, Q6 to Q9, R30 to R10, R7 to R16, R1 to R18, R2 to R19, R8 to R21, R31 to R3, R52 to R30, R56 to R31, R54 to R32, R58 to R33, R38 to R35, R40 to R37, R53 to R38, R57 to R39, R55 to R40, R59 to R41, R35 to R42, R39 to R43, R37 to R44, R41 to R45, R29 to R5, R26 to R6, R23 to R7, R27 to R8, R24 to R9
Connections:
- net +3.3V: now also R11.1, R12.1, R13.1, R14.1, R17.1, R20.1, R22.1, R23.1, R24.1, R25.1, R26.1, R27.1, R28.1, R29.1; no longer U1.9 (V_{DD})
- net GND: now also J4.1 (Pin_1), D2.1 (K), D4.1 (K); no longer J4.5 (Pin_5)
- net at A1.24 (SCL/A5), U1.12 (SCK): now also R20.2
- net at J7.1 (Pin_1), U1.25 (GPA4): now also D14.1 (K)
- net at J7.2 (Pin_2), U1.26 (GPA5): now also D15.1 (K)
- net at J7.3 (Pin_3), U1.27 (GPA6): now also D16.1 (K)
- net at J7.4 (Pin_4), U1.28 (GPA7): now also D17.1 (K)
- net at A1.10 (D7): now also R6.1, R2.1; no longer J2.2 (Pin_2)
- net at A1.11 (D8): now also R5.1, R1.1; no longer J2.1 (Pin_1)
- net at J5.1 (Pin_1), Q4.1 (C): now also A1.25 (A6); no longer A1.19 (A0)
- net at A1.20 (A1): now also J4.3 (Pin_3); no longer J4.1 (Pin_1)
- net at J4.2 (Pin_2): now also A1.19 (A0); no longer A1.21 (A2)
- net at A1.22 (A3): now also J4.5 (Pin_5); no longer J4.3 (Pin_3)
- net at A1.23 (SDA/A4), U1.13 (SDA): now also R17.2
- net at J4.4 (Pin_4): now also A1.21 (A2); no longer A1.25 (A6)
- net at A1.5 (D2): now also J2.4 (Pin_4), D8.1 (K); no longer R7.1
- net at A1.6 (D3): now also J2.3 (Pin_3), D7.1 (K); no longer R6.1
- net at A1.7 (D4): now also J2.2 (Pin_2), D6.1 (K); no longer R5.1
- net at A1.8 (D5): now also J2.1 (Pin_1), D5.1 (K); no longer J2.4 (Pin_4)
- net at A1.9 (D6): now also R7.1, R4.1; no longer J2.3 (Pin_3)
- net at J6.3 (Pin_3), U1.23 (GPA2): now also D12.1 (K)
- net at J6.1 (Pin_1), U1.21 (GPA0): now also D10.1 (K)
- net at J6.2 (Pin_2), U1.22 (GPA1): now also D11.1 (K)
- net at J6.4 (Pin_4), U1.24 (GPA3): now also D13.1 (K)
- net at D1.2 (A): now also R1.2
- new net: D11.2 (A), R23.2
- new net: D7.2 (A), R13.2
- new net: D2.2 (A), R2.2
- new net: D6.2 (A), R12.2
- new net: D16.2 (A), R28.2
- new net: D8.2 (A), R14.2
- new net: D4.2 (A), R4.2
- new net: D17.2 (A), R29.2
- new net: D5.2 (A), R11.2
- new net: D10.2 (A), R22.2
- new net: D14.2 (A), R26.2
- new net: D13.2 (A), R25.2
- new net: D12.2 (A), R24.2
- new net: D15.2 (A), R27.2
Other:
- moved on the sheet: A1, C1, C2, D1, D18, D19, D20, D21, D22, D23, D24, D25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
